File: projects/kart-medulla/kart-medulla_P1.kicad_sch (KiCad schematic)
At the start: 55 parts, among them CN1 1990012, CN10 1990012, CN2 1990012, CN3 1990012, CN4 1990012, CN5 1990012, CN6 1990012, CN7 1990012, CN8 1990012, CN9 1990012, Q3 IRLZ44NPBF, Q4 BSS123_C5184436, U1 LM358DR, U13 MCP4922-E/SL, U14 MAX4660EUA+T, U19 L7805CDT_C20611927, U23 SSW-122-01-T-D, U24 SSW-122-01-T-S, U25 PCF8574T/3,518, U5 SN74LVC3G17DCTR

Commit message: kart-medulla: cluster U25 signals on right side (6-label reshuffle)
U25 (PCF8574 GPIO expander) physically placed near CN3. Re-clustered
all U25-facing signals on right-side CNs to minimize routing length:
- CN3 now pure EXP cluster (P1/P2/P3)
- CN4 carries REVERSE_WIRE + I²C (SDA/SCL) — all U25 control
- Displaced ESP32 signals (CMD_STEER_DIR/PWM, SDC_IN_LOW_SIDE) moved
  to left CNs (CN8/CN9), where their ESP32 GPIOs cross under the
  module via the bottom layer.

6 net-label renames on the CN-side; no wire/footprint geometry
changed. Verified end-to-end via netlist export + ERC clean.

pinout-cn-connectors.md and history.md updated accordingly.

Co-Authored-By: Claude Opus 4.7 (1M context) <noreply@anthropic.com>
Connections:
- net CMD_STEER_DIR__3V3: now also CN8.3; no longer CN3.1
- net CMD_STEER__PWM_3V3: now also CN9.1; no longer CN4.3
- net EXP_P3: now also CN3.1; no longer CN8.3
- net SCL__I2C: now also CN4.3; no longer CN9.1
- net SDA__I2C: now also CN4.2; no longer CN8.1
- net SDC_IN_LOW_SIDE: now also CN8.1; no longer CN4.2
Changed lines of the file:
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@@
 		)
 	)
-	(label "SDA__I2C"
+	(label "SDC_IN_LOW_SIDE"
 		(at 163.83 62.23 0)
 		(effects
@@
 		)
 	)
-	(label "SCL__I2C"
+	(label "CMD_STEER__PWM_3V3"
 		(at 163.83 78.74 0)
 		(effects
@@
 		)
 	)
-	(label "CMD_STEER__PWM_3V3"
+	(label "SCL__I2C"
 		(at 100.33 52.07 0)
 		(effects
@@
 		)
 	)
-	(label "CMD_STEER_DIR__3V3"
+	(label "EXP_P3"
 		(at 45.72 80.01 0)
 		(effects
@@
 		)
 	)
-	(label "SDC_IN_LOW_SIDE"
+	(label "SDA__I2C"
 		(at 100.33 49.53 0)
 		(effects
@@
 		)
 	)
-	(label "EXP_P3"
+	(label "CMD_STEER_DIR__3V3"
 		(at 163.83 67.31 0)
 		(effects

Commit message: kart-medulla: swap CN5.3 GND ↔ CN9.3 EXP_P4
EXP_P4 was the last U25-related signal still on a left-side CN after
yesterday's cluster reshuffle. Moved to CN5.3 (right) so all four
PCF8574 expander outputs (P1–P4) sit on right-side CNs near U25.
GND moves to CN9.3 in its place.

Co-Authored-By: Claude Opus 4.7 (1M context) <noreply@anthropic.com>
Connections:
- net EXP_P4: now also CN5.3; no longer CN9.3
- net GND: now also CN9.3; no longer CN5.3
Changed lines of the file:
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@@
 		)
 	)
-	(label "GND"
+	(label "EXP_P4"
 		(at 100.33 67.31 0)
 		(effects
@@
 		)
 	)
-	(label "EXP_P4"
+	(label "GND"
 		(at 163.83 83.82 0)
 		(effects
