File: projects/kart-medulla/kart-medulla.kicad_pcb (KiCad board)
At the start: 2 copper layers, 68.9 x 66.5 mm, 59 parts, among them CN1 1990012, CN10 1990012, CN2 1990012, CN3 1990012, CN4 1990012, CN5 1990012, CN6 1990012, CN7 1990012, CN8 1990012, CN9 1990012, Q3 IRLZ44NPBF, Q4 BSS123_C5184436, U1 LM358DR, U13 MCP4922-E/SL, U14 MAX4660EUA+T, U19 L7805CDT_C20611927, U23 SSW-122-01-T-D, U24 SSW-122-01-T-S, U25 PCF8574T/3,518, U5 SN74LVC3G17DCTR

Commit message: pcb in progress
Parts:
- moved R8 131.1 mm to (133.9, 45.7), turned to 0 degrees
- moved R9 126.6 mm to (130.6, 45.7), turned to 180 degrees
- moved R31 125.7 mm to (141.0, 67.9), turned to 0 degrees
- moved R30 125.6 mm to (141.0, 69.8)
- moved R26 124.6 mm to (125.0, 51.8), turned to 90 degrees
- moved R10 122.1 mm to (127.3, 45.7), turned to 180 degrees
- moved R27 121.0 mm to (125.0, 54.9)
- moved Q4 120.5 mm to (141.0, 64.8), turned to -90 degrees
- moved R17 101.8 mm to (89.7, 54.4)
- moved R15 101.1 mm to (89.9, 50.8)
- moved R16 98.3 mm to (87.1, 54.4), turned to 90 degrees
- moved R14 97.8 mm to (87.1, 50.8)
- moved R20 90.3 mm to (87.8, 101.7), turned to 90 degrees
- moved U1 89.9 mm to (82.5, 100.3), turned to -90 degrees
- moved C5 87.2 mm to (69.1, 53.1), turned to -90 degrees
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Connections:
- CN1 pad 1: GND -> +3V3
- CN3 pad 2: /P1/EXP_P1 -> /P1/EXP_P2
- CN3 pad 3: /P1/EXP_P2 -> /P1/EXP_P1
- CN5 pad 3: GND -> /P1/EXP_P4
- CN6 pad 1: /P1/PEDAL_ACC__0_5V -> /P1/PEDAL_BRAKE__0_5V
- CN6 pad 2: /P1/PEDAL_BRAKE__0_5V -> /P1/PEDAL_ACC__0_5V
- CN9 pad 3: /P1/EXP_P4 -> GND
- U23 pad 19: unconnected-(U23-Pad19) -> /P1/CMD_STEER_DIR__3V3
- U23 pad 20: unconnected-(U23-Pad20) -> /P1/CMD_STEER_DIR__3V3
- U23 pad 21: unconnected-(U23-Pad21) -> /P1/SDC_NOT_EMERGENCY__3V3
- U23 pad 22: unconnected-(U23-Pad22) -> /P1/SDC_NOT_EMERGENCY__3V3
- U24 pad 13: /P1/SDC_NOT_EMERGENCY__3V3 -> unconnected-(U24-Pad13)
- U24 pad 9: /P1/CMD_STEER_DIR__3V3 -> unconnected-(U24-Pad9)
Routing:
- net +5V_REG: track 0.00 -> 76.6 mm
- net +12V: track 0.00 -> 72.3 mm
- net +3V3: track 0.00 -> 71.8 mm
- net /P1/SDA__I2C: track 0.00 -> 37.9 mm
- net /P1/SCL__I2C: track 0.00 -> 35.8 mm
- net /P1/MOTOR_HALL_3__3V3: track 0.00 -> 32.1 mm
- net /P1/EXP_P2: track 0.00 -> 30.9 mm
- net /P1/MOTOR_HALL_2__3V3: track 0.00 -> 29.3 mm
- net /P1/EXP_P4: track 0.00 -> 28.5 mm
- net /P1/EXP_P3: track 0.00 -> 27.4 mm
- net /P1/BUZZER: track 0.00 -> 25.2 mm
- net /P1/EXP_P1: track 0.00 -> 24.9 mm
- net /P1/PEDAL_ACC__0_5V: track 0.00 -> 24.3 mm
- net /P1/PRESSURE_1__0_10V: track 0.00 -> 24.1 mm
- net /P1/CMD_STEER_DIR__3V3: track 0.00 -> 18.1 mm
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Other:
- board outline removed
- board text removed: "POWER"

Commit message: pcb in progress
Parts:
- moved R22 12.8 mm to (74.2, 67.8), turned to 0 degrees
- moved R23 6.82 mm to (70.4, 67.8), turned to 0 degrees
- turned Q3 to 0 degrees
Routing:
- net +3V3: track 71.8 -> 146.0 mm
- net +5V_REG: track 76.6 -> 136.0 mm
- net /P1/SDC_NOT_EMERGENCY__3V3: track 5.61 -> 23.8 mm
- net /P1/HYDRAULIC_1__0_5V: track 0.00 -> 13.0 mm
- net /P1/SDC_IN_LOW_SIDE: track 11.0 -> 0.14 mm
- net /P1/HYDRAULIC_1__0_3V3: track 0.00 -> 10.8 mm
- net Net-(Q3-G): track 7.99 -> 6.94 mm

Commit message: pcb routes update
Routing:
- net /P1/MOTOR_HALL_1__3V3: track 0.00 -> 123.5 mm
- net /P1/MOTOR_HALL_1__5V: track 0.00 -> 103.1 mm
- net /P1/CMD_ACC__0_5V: track 0.00 -> 49.3 mm
- net /P1/CMD_STEER__PWM_3V3: track 0.00 -> 48.1 mm
- net /P1/CMD_ACC_ESP32__0_5V: track 0.00 -> 46.0 mm
- net /P1/SDC_IN_LOW_SIDE: track 0.14 -> 11.0 mm
- net /P1/CMD_BRAKE__0_5V: track 12.4 -> 22.1 mm
- net +5V_REG: track 136.0 -> 140.8 mm

Commit message: refilled update
Parts:
- moved PAD2 17.9 mm to (157.0, 102.0)
- moved PAD4 11.4 mm to (152.0, 47.0)
- moved PAD1 6.98 mm to (65.6, 102.0)
- moved PAD3 5.00 mm to (62.0, 44.0)
- moved CN4 2.74 mm to (132.0, 62.5), turned to -90 degrees
- moved CN3 2.65 mm to (132.0, 72.5), turned to -90 degrees
Connections:
- CN3 pad 1: /P1/EXP_P3 -> /P1/EXP_P1
- CN3 pad 3: /P1/EXP_P1 -> /P1/EXP_P3
- CN4 pad 1: /P1/REVERSE_WIRE -> /P1/SCL__I2C
- CN4 pad 3: /P1/SCL__I2C -> /P1/REVERSE_WIRE
Routing:
- net /P1/SCL__I2C: track 35.8 -> 77.6 mm
- net /P1/SDA__I2C: track 37.9 -> 76.0 mm
- net /P1/SELECT_THROTTLE: track 2.44 -> 32.5 mm, vias 0 -> 1
- net /P1/CMD_STEER__PWM_3V3: track 48.1 -> 60.9 mm
- net /P1/EXP_P2: track 30.9 -> 23.2 mm
- net /P1/REVERSE_WIRE: track 8.90 -> 12.0 mm
- net /P1/EXP_P3: track 27.4 -> 30.0 mm
- net /P1/EXP_P1: track 24.9 -> 25.7 mm
- removed copper zone on F.Cu, net GND
Other:
- board outline added: 107 x 90.1 mm
